File: schematic_pcb/USB-C Meter.kicad_pcb (KiCad board)
At the start: 2 copper layers, 58.5 x 48 mm, 11 parts, among them J1 USB_C_Receptacle_PowerOnly_6P, J2 USB_C_Receptacle_PowerOnly_6P, U1 WEMOS_D1_mini, U2 INA226, U3 Display I2C

Commit message: fix: updated schematic and pcb to version 1.2
Parts:
- removed C4: 0.1µ, Capacitor_SMD:C_0603_1608Metric
- added C1: 0.1µ, Capacitor_SMD:C_0603_1608Metric, F.Cu at (87.5, 57.5)
- added R2: 10, Resistor_SMD:R_0603_1608Metric_Pad0.98x0.95mm_HandSolder, F.Cu at (86.5, 60.5)
- added R3: 10, Resistor_SMD:R_0603_1608Metric_Pad0.98x0.95mm_HandSolder, F.Cu at (88.5, 60.5)
- added REF**: MountingHole_2.2mm_M2_DIN965_Pad, MountingHole:MountingHole_2.2mm_M2_DIN965_Pad, F.Cu at (71.5, 72.5)
- added REF**: MountingHole_2.2mm_M2_DIN965_Pad, MountingHole:MountingHole_2.2mm_M2_DIN965_Pad, F.Cu at (65.5, 34.0)
- added REF**: MountingHole_2.2mm_M2_DIN965_Pad, MountingHole:MountingHole_2.2mm_M2_DIN965_Pad, F.Cu at (109.5, 34.0)
- added REF**: MountingHole_2.2mm_M2_DIN965_Pad, MountingHole:MountingHole_2.2mm_M2_DIN965_Pad, F.Cu at (103.5, 72.5)
- C2: footprint Capacitor_Tantalum_SMD:CP_EIA-6032-20_AVX-F -> Capacitor_Tantalum_SMD:CP_EIA-7343-30_AVX-N
- R4, R5: footprint Resistor_SMD:R_0402_1005Metric -> Resistor_SMD:R_0603_1608Metric_Pad0.98x0.95mm_HandSolder
- moved C2 26.7 mm to (88.0, 37.0), turned to 0 degrees
- moved C3 3.61 mm to (87.5, 52.0)
- moved J2 2.00 mm to (111.0, 67.5)
- moved R5 1.58 mm to (87.5, 50.5)
- moved J1 1.50 mm to (64.0, 67.5)
- moved R4 1.12 mm to (87.5, 49.0)
- moved U2 0.50 mm to (87.5, 55.0)
Connections:
- net Net-(J1-SHIELD) renamed GND
- net Net-(U1-3V3) renamed 3V3
- J1 pad A9: Net-(U2-Vin+) -> /VBUS1
- J1 pad B9: Net-(U2-Vin+) -> /VBUS1
- J2 pad A9: Net-(U2-Vbus) -> /VBUS2
- J2 pad B9: Net-(U2-Vbus) -> /VBUS2
- R1 pad 1: Net-(U2-Vin+) -> /VBUS1
- R1 pad 2: Net-(U2-Vbus) -> /VBUS2
Routing:
- net Net-(U2-Vbus): track 41.1 -> 7.75 mm
- net Net-(U2-Vin+): track 36.9 -> 3.95 mm
- net /VBUS1: track 0.00 -> 30.1 mm
- net /VBUS2: track 0.00 -> 29.5 mm
- net 3V3: track 57.0 -> 32.9 mm
- net GND: track 70.5 -> 53.0 mm
- net Net-(J1-CC2): track 44.6 -> 41.1 mm
- net Net-(J1-CC1): track 44.6 -> 41.1 mm
- net Net-(U1-SDA/D2): track 27.1 -> 26.0 mm
- added copper zone on F.Cu, net /VBUS1
- added copper zone on F.Cu, net /VBUS2
Other:
- board size 58.5 x 48 mm -> 54 x 48 mm
- board text added: "MacWake USB-C Meter V1.2"
- board text removed: "MacWake USB-C Meter V1.1"
