File: schematic_pcb/USB-C Meter.kicad_sch (KiCad schematic)
At the start: 11 parts, among them J1 USB_C_Receptacle_PowerOnly_6P, J2 USB_C_Receptacle_PowerOnly_6P, U1 WEMOS_D1_mini, U2 INA226, U3 Display I2C

Commit message: fix: updated schematic and pcb to version 1.2
Parts:
- removed C4: 0.1µ, Capacitor_SMD:C_0603_1608Metric, symbol Device:C
- added C1: 0.1µ, Capacitor_SMD:C_0603_1608Metric, symbol Device:C
- added R2, R3: 10, Resistor_SMD:R_0603_1608Metric_Pad0.98x0.95mm_HandSolder, symbol Device:R
- C2: footprint Capacitor_Tantalum_SMD:CP_EIA-6032-20_AVX-F -> Capacitor_Tantalum_SMD:CP_EIA-7343-30_AVX-N; symbol PCM_Capacitor_AKL:CP_SMD_Tantalum_AVX-F_6032 -> Device:C_Polarized
- R4, R5: footprint Resistor_SMD:R_0402_1005Metric -> Resistor_SMD:R_0603_1608Metric_Pad0.98x0.95mm_HandSolder
Connections:
- net VBUS1: now reaches J1.A9 (VBUS), J1.B9 (VBUS), R1.1
- net VBUS1: now also R2.2; no longer U2.10 (Vin+)
- net 3V3: now reaches C2.1, C3.1, R4.2, R5.2, U1.8 (3V3), U2.2 (A0), U2.6 (VS), U3.1 (VDD)
- net at U2.8 (Vbus), U2.9 (Vin-): now also C1.2, R3.1
- net VBUS2: now reaches J2.A9 (VBUS), J2.B9 (VBUS), R1.2
- net VBUS2: now also R3.2
- new net: C1.1, R2.1, U2.10 (Vin+)
- no-connect marks 0 -> 13
Other:
- moved on the sheet: U1
